File: MainBoard/MainBoard.kicad_pcb (KiCad board)
At the start: 2 copper layers, 45 parts, among them J1 Conn_01x01, J2 Conn_01x01, J3 Conn_01x04, J4 Conn_01x01, J5 RJ45, J6 RJ12, Q1 PN2222A, Q2 PN2222A, Q3 PN2222A, Q4 PN2222A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

Commit message: List Components
Parts:
- moved J6 121.6 mm to (59.7, 132.7)
- moved J5 99.4 mm to (64.8, 92.7)
- moved J4 98.2 mm to (257.8, 50.8)
- moved U1 71.3 mm to (220.3, 54.0)
- moved SW1 62.8 mm to (159.4, 159.4)
- moved J1 43.3 mm to (174.0, 146.1)
- moved J3 40.5 mm to (257.8, 55.9)
- moved J2 29.3 mm to (269.9, 121.9)
- moved D1 11.8 mm to (156.2, 146.1)
Changed lines of the file:
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@@
     (links 83)
     (no_connects 83)
-    (area 0 0 0 0)
+    (area 157.48 87.63 253.450002 143.265239)
     (thickness 1.6)
     (drawings 0)
@@
   )
   (module std_lib_SRC:Diode (layer F.Cu)
-    (at 158.955001 134.555)
+    (at 156.21 146.05)
     (descr "D, pin pitch=12.7mm")
     (tags diode)
@@
   )
   (module std_lib_SRC:CONN_1x01 (layer F.Cu)
-    (at 213.775 129.02762)
+    (at 173.99 146.05)
     (descr "Low profile, screw machine socket strip, through hole, 100mil / 2.54mm pitch")
     (tags connector)
@@
   )
   (module std_lib_SRC:CONN_1x01 (layer F.Cu)
-    (at 242.245 112.31762)
+    (at 269.875 121.92)
     (descr "Low profile, screw machine socket strip, through hole, 100mil / 2.54mm pitch")
     (tags connector)
@@
   )
   (module std_lib_SRC:CONN_1x04 (layer F.Cu)
-    (at 235.345 89.625001)
+    (at 257.81 55.88)
     (descr "Low profile, screw machine socket strip, through hole, 100mil / 2.54mm pitch")
     (tags connector)
@@
   )
   (module std_lib_SRC:CONN_1x01 (layer F.Cu)
-    (at 213.775 138.51762)
+    (at 257.81 50.8)
     (descr "Low profile, screw machine socket strip, through hole, 100mil / 2.54mm pitch")
     (tags connector)
@@
   )
   (module std_lib_SRC:RJ45_8_Shield (layer F.Cu)
-    (at 161.265001 116.525001)
+    (at 64.77 92.71)
     (tags RJ45)
     (fp_text reference J5 (at 4.7 11.18) (layer F.SilkS)
@@
   )
   (module std_lib_SRC:RJ_12 (layer F.Cu)
-    (at 174.465001 92.675001)
+    (at 59.69 132.715)
     (tags RJ_12)
     (fp_text reference J6 (at 3.3 6.35) (layer F.SilkS)
@@
   )
   (module std_lib_SRC:DIP-4_W7.62mm (layer F.Cu)
-    (at 206.375001 117.675)
+    (at 159.385 159.385)
     (descr "4-lead dip package, row spacing 7.62 mm (300 mils)")
     (tags "DIP 7.62mm Socket")
@@
   )
   (module std_lib_SRC:DIP-16_W7.62mm (layer F.Cu)
-    (at 159.405001 90.995)
+    (at 220.345 53.975)
     (descr "16-lead dip package, row spacing 7.62 mm (300 mils), Socket")
     (tags "DIP 7.62mm Socket")
