File: SideBoard/SideBoard.sch (KiCad schematic (older format))
At the start: 22 parts, among them J1 RJ45, J2 RJ12

Commit message: Correct mistakes on SideBoard + begin routing
Parts:
- removed D7: LED, std_lib_SRC:LED_D5.0mm, symbol LED
- removed D8: 1N4148, std_lib_SRC:Diode, symbol D
- D5: footprint std_lib_SRC:Resistor -> std_lib_SRC:LED_D5.0mm
- renumbered D12 to D10, D13 to D11, D14 to D12, D15 to D13, D16 to D14, D17 to D15, D18 to D16, D19 to D17, D20 to D18, D9 to D7, D10 to D8, D11 to D9
Other:
- moved on the sheet: D10, D11, D12, D13, D14, D15, D16, D17, D18, D7, D8, D9
Changed lines of the file:
@@
 F 0 "D5" H 4900 1950 50  0000 C CNN
 F 1 "LED" H 4900 1750 50  0000 C CNN
-F 2 "std_lib_SRC:Resistor" H 4900 1850 50  0001 C CNN
+F 2 "std_lib_SRC:LED_D5.0mm" H 4900 1850 50  0001 C CNN
 F 3 "" H 4900 1850 50  0001 C CNN
 	1    4900 1850
@@
 $Comp
 L LED D7
-U 1 1 5B3B7D96
+U 1 1 5B3B7E3E
 P 4900 2450
 F 0 "D7" H 4900 2550 50  0000 C CNN
@@
 $Comp
 L D D8
-U 1 1 5B3B7D9C
+U 1 1 5B3B7E44
 P 4900 2750
 F 0 "D8" H 4900 2850 50  0000 C CNN
@@
 $EndComp
 Text GLabel 4550 2450 0    60   Input ~ 0
-P3
+P4
 $Comp
 L LED D9
-U 1 1 5B3B7E3E
+U 1 1 5B3B7F16
 P 4900 3050
 F 0 "D9" H 4900 3150 50  0000 C CNN
@@
 $Comp
 L D D10
-U 1 1 5B3B7E44
+U 1 1 5B3B7F1C
 P 4900 3350
 F 0 "D10" H 4900 3450 50  0000 C CNN
@@
 $EndComp
 Text GLabel 4550 3050 0    60   Input ~ 0
-P4
+P5
 $Comp
 L LED D11
-U 1 1 5B3B7F16
+U 1 1 5B3B7FE6
 P 4900 3650
 F 0 "D11" H 4900 3750 50  0000 C CNN
@@
 $Comp
 L D D12
-U 1 1 5B3B7F1C
+U 1 1 5B3B7FEC
 P 4900 3950
 F 0 "D12" H 4900 4050 50  0000 C CNN
@@
 $EndComp
 Text GLabel 4550 3650 0    60   Input ~ 0
-P5
+P6
 $Comp
 L LED D13
-U 1 1 5B3B7FE6
+U 1 1 5B3B80BE
 P 4900 4250
 F 0 "D13" H 4900 4350 50  0000 C CNN
@@
 $Comp
 L D D14
-U 1 1 5B3B7FEC
+U 1 1 5B3B80C4
 P 4900 4550
 F 0 "D14" H 4900 4650 50  0000 C CNN
@@
 $EndComp
 Text GLabel 4550 4250 0    60   Input ~ 0
-P6
+P7
 $Comp
 L LED D15
-U 1 1 5B3B80BE
+U 1 1 5B3B81A2
 P 4900 4850
 F 0 "D15" H 4900 4950 50  0000 C CNN
@@
 $Comp
 L D D16
-U 1 1 5B3B80C4
+U 1 1 5B3B81A8
 P 4900 5150
 F 0 "D16" H 4900 5250 50  0000 C CNN
@@
 $EndComp
 Text GLabel 4550 4850 0    60   Input ~ 0
-P7
+P8
 $Comp
 L LED D17
-U 1 1 5B3B81A2
+U 1 1 5B3B82C6
 P 4900 5450
 F 0 "D17" H 4900 5550 50  0000 C CNN
@@
 $Comp
 L D D18
-U 1 1 5B3B81A8
+U 1 1 5B3B82CC
 P 4900 5750
 F 0 "D18" H 4900 5850 50  0000 C CNN
@@
 $EndComp
 Text GLabel 4550 5450 0    60   Input ~ 0
-P8
-$Comp
-L LED D19
-U 1 1 5B3B82C6
-P 4900 6050
-F 0 "D19" H 4900 6150 50  0000 C CNN
-F 1 "LED" H 4900 5950 50  0000 C CNN
-F 2 "std_lib_SRC:LED_D5.0mm" H 4900 6050 50  0001 C CNN
-F 3 "" H 4900 6050 50  0001 C CNN
-	1    4900 6050
-	-1   0    0    1
-$EndComp
-$Comp
-L D D20
-U 1 1 5B3B82CC
-P 4900 6350
-F 0 "D20" H 4900 6450 50  0000 C CNN
-F 1 "1N4148" H 4900 6250 50  0000 C CNN
-F 2 "std_lib_SRC:Diode" H 4900 6350 50  0001 C CNN
-F 3 "" H 4900 6350 50  0001 C CNN
-	1    4900 6350
-	1    0    0    -1
-$EndComp
-Text GLabel 4550 6050 0    60   Input ~ 0
 P9
 Wire Wire Line
@@
 	5050 650  5150 650
 Wire Wire Line
-	5150 650  5150 6350
-Wire Wire Line
 	5150 950  5050 950
 Wire Wire Line
@@
 	4650 5750 4650 5450
 Connection ~ 4650 5450
-Wire Wire Line
-	4550 6050 4750 6050
-Wire Wire Line
-	5150 6050 5050 6050
-Wire Wire Line
-	5150 6350 5050 6350
-Wire Wire Line
-	4750 6350 4650 6350
-Wire Wire Line
-	4650 6350 4650 6050
-Connection ~ 4650 6050
 Connection ~ 5150 1250
 Connection ~ 5150 950
 Connection ~ 5150 1850
 Connection ~ 5150 1550
+Connection ~ 5150 2150
 Connection ~ 5150 2450
-Connection ~ 5150 2150
 Connection ~ 5150 3050
 Connection ~ 5150 2750
@@
 Connection ~ 5150 5450
 Connection ~ 5150 5150
-Connection ~ 5150 6050
-Connection ~ 5150 5750
+Wire Wire Line
+	5150 650  5150 5750
 $EndSCHEMATC
